Commit message: YAM teleop integration: real-arm-accurate model + grasp tool frame
- EE frame fix: use real link6 (from i2rt combined yam+linear_4310) plus a
  `grasp` tool frame matching i2rt's grasp_site (link_name="grasp", +Z=approach).
  The standalone yam.xml link6 was a placeholder i2rt overrides via the gripper mount.
- Generate consistent yam.urdf from yam.xml (scripts/gen_yam_urdf.py).
- Complete MJCF for sim: position actuators, home keyframe, link6 mass,
  armature/damping, visual-only geoms.
- scene.xml: right_target mocap gizmo (vis_target).
- Stock full-pose teleop (scripts/teleop_yam_mujoco.py) + IK/joint/orient tests.
- skills/adding-a-new-arm: the EE tool-frame gotcha + recipe.
- Orin setup/status docs + helper scripts.

Co-Authored-By: Claude Opus 4.8 <noreply@anthropic.com>

File: assets/yam/yam.urdf (robot description, URDF)
Before this commit: robot yam_v0, 7 links, 6 joints
Links:
- removed link link_1
- removed link link_2
- removed link link_3
- removed link link_4
- removed link link_5
- removed link link_6
- added link grasp, mass 0.5
- added link link1, mass 0.5
- added link link2, mass 0.5
- added link link3, mass 0.5
- added link link4, mass 0.5
- added link link5, mass 0.5
- added link link6, mass 0.5
- link base_link: mass 0.822546 -> None; geometry 
Joints:
- added joint fixed_grasp: type fixed, parent link6, child grasp, origin xyz=0.000000000 0.000000000 -0.134700000 rpy=3.141592654 -0.000000000 0.000000000
- joint joint1: axis 0 0 1 -> 0.000000 0.000000 1.000000; child link_1 -> link1; limit lower=-2.61799 upper=3.13 effort=10 velocity=10 -> lower=-2.617990 upper=3.054330 effort=100 velocity=3.14159; origin xyz=-3.55271e-18 -1.05495e-18 0.0631 rpy=0 -0 1.5708 -> xyz=0.000000000 0.000000000 0.067000000 rpy=0.000000000 0.000000000 -1.570800569
- joint joint2: axis 0 0 1 -> 0.000000 0.000000 1.000000; child link_2 -> link2; limit lower=0 upper=3.65 effort=10 velocity=10 -> lower=0.000000 upper=3.650000 effort=100 velocity=3.14159; origin xyz=2.5e-05 -0.02 0.0409 rpy=1.5708 -1.98004e-28 1.5708 -> xyz=-0.032900000 0.020000000 0.045500000 rpy=1.570800327 0.000000000 -1.570800327; parent link_1 -> link1
- joint joint3: axis 0 0 1 -> 0.000000 0.000000 1.000000; child link_3 -> link3; limit lower=0 upper=3.13 effort=10 velocity=10 -> lower=0.000000 upper=3.665190 effort=100 velocity=3.14159; origin xyz=0.264 0 6.77626e-21 rpy=-3.14159 1.26218e-29 7.88861e-31 -> xyz=0.264000000 0.000000408 -0.063750000 rpy=-3.141590000 -0.000000000 1.570800569; parent link_2 -> link2
- joint joint4: axis 0 0 1 -> 0.000000 0.000000 1.000000; child link_4 -> link4; limit lower=-1.5708 upper=1.5708 effort=10 velocity=10 -> lower=-1.570800 upper=1.570800 effort=100 velocity=3.14159; origin xyz=-0.245 -0.0600003 -1.9984e-15 rpy=-5.65471e-31 -1.1507e-13 2.94252e-43 -> xyz=0.060000300 -0.244999000 -0.002050000 rpy=0.000000000 0.000000000 -3.141590000; parent link_3 -> link3
- joint joint5: axis 0 0 1 -> 0.000000 0.000000 1.000000; child link_5 -> link5; limit lower=-1.5708 upper=1.5708 effort=10 velocity=10 -> lower=-1.570800 upper=1.570800 effort=100 velocity=3.14159; origin xyz=-0.0739968 -0.0395003 2.44738e-05 rpy=-1.5708 1.5708 0 -> xyz=-0.040300300 0.070385100 -0.032388700 rpy=0.000002327 -1.570792084 -3.141592327; parent link_4 -> link4
- joint joint6: axis 0 0 1 -> 0.000000 0.000000 -1.000000; child link_6 -> link6; limit lower=-2.0944 upper=2.0944 effort=10 velocity=10 -> lower=-2.094400 upper=2.094400 effort=100 velocity=3.14159; origin xyz=-4.0742e-16 0.0353 0.0395 rpy=-1.5708 3.81639e-16 4.68582e-15 -> xyz=0.000000240 -0.041948100 0.040499600 rpy=1.570794327 -1.570792327 3.141590654; parent link_5 -> link5
